Commit message: wheel align

File: model/Sagan.xacro.urdf (robot description, URDF)
Before this commit: robot Sagan, 12 links, 11 joints
Joints:
- joint LF_stering_arm_joint: origin xyz=-0.185 -0.031 0.04225 rpy=0 -1.5068 0 -> xyz=-0.185 -0.031 0.04225 rpy=0 -1.5708 0
- joint LR_stering_arm_joint: origin xyz=0.185 -0.031 0.04225 rpy=0 1.5683 0 -> xyz=0.185 -0.031 0.04225 rpy=0 1.5708 0
- joint RF_stering_arm_joint: origin xyz=0.185 -0.031 0.04225 rpy=3.1416 1.5372 3.1416 -> xyz=0.185 -0.031 0.04225 rpy=3.1416 1.5708 3.1416
- joint RR_stering_arm_joint: origin xyz=-0.185 -0.031 0.04225 rpy=0 -1.3763 0 -> xyz=-0.185 -0.031 0.04225 rpy=0 -1.5708 0

Commit message: rviz2 no loading meshes issue solved

File: model/Sagan.xacro.urdf (robot description, URDF)
Before this commit: robot Sagan, 12 links, 11 joints
Links:
- link LF_stering_arm: geometry collision mesh filename=file://$(find sagan_description)/model/meshes/LF_stering_ar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; visual mesh filename=file://$(find sagan_description)/model/meshes/LF_stering_ar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
- link LF_wheel: geometry collision mesh filename=file://$(find sagan_description)/model/meshes/LF_wheel.STL; visual mesh filename=file://$(find sagan_description)/model/meshes/LF_wheel.STL
- link LR_stering_arm: geometry collision mesh filename=file://$(find sagan_description)/model/meshes/LR_stering_ar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; visual mesh filename=file://$(find sagan_description)/model/meshes/LR_stering_ar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
- link LR_wheel: geometry collision mesh filename=file://$(find sagan_description)/model/meshes/LR_wheel.STL; visual mesh filename=file://$(find sagan_description)/model/meshes/LR_wheel.STL
- link Left_arm: geometry collision mesh filename=file://$(find sagan_description)/model/meshes/Left_arm.STL; visual mesh filename=file://$(find sagan_description)/model/meshes/Left_arm.STL
- link RF_stering_arm: geometry collision mesh filename=file://$(find sagan_description)/model/meshes/RF_stering_ar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; visual mesh filename=file://$(find sagan_description)/model/meshes/RF_stering_ar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
- link RF_wheel: geometry collision mesh filename=file://$(find sagan_description)/model/meshes/RF_wheel.STL; visual mesh filename=file://$(find sagan_description)/model/meshes/RF_wheel.STL
- link RR_stering_arm: geometry collision mesh filename=file://$(find sagan_description)/model/meshes/RR_stering_ar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; visual mesh filename=file://$(find sagan_description)/model/meshes/RR_stering_ar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
- link RR_wheel: geometry collision mesh filename=file://$(find sagan_description)/model/meshes/RR_wheel.STL; visual mesh filename=file://$(find sagan_description)/model/meshes/RR_wheel.STL
- link Right_arm: geometry collision mesh filename=file://$(find sagan_description)/model/meshes/Right_arm.STL; visual mesh filename=file://$(find sagan_description)/model/meshes/Right_arm.STL
- link base_link: geometry collision mesh filename=file://$(find sagan_description)/model/meshes/base_link.STL; visual mesh filename=file://$(find sagan_description)/model/meshes/base_link.STL
Joints:
- removed joint base_link_joint
- added joint base_footprint_joint: type fixed, parent base_footprint, child base_link, origin xyz=0 0 0.017 rpy=-1.5708 0 0

Commit message: wheels joints orientation fixed

File: model/Sagan.xacro.urdf (robot description, URDF)
Before this commit: robot Sagan, 12 links, 11 joints
Joints:
- joint RF_wheel_joint: axis 0 0 1 -> 0 0 -1
- joint RR_wheel_joint: axis 0 0 1 -> 0 0 -1

Commit message: Sterring joints added to controllers parameters

File: model/Sagan.xacro.urdf (robot description, URDF)
Before this commit: robot Sagan, 12 links, 11 joints
Joints:
- joint LF_stering_arm_joint: type fixed -> continuous
- joint LR_stering_arm_joint: type fixed -> continuous
- joint RF_stering_arm_joint: type fixed -> continuous
- joint RR_stering_arm_joint: type fixed -> continuous

File: model/ros2_control.xacro (robot description, xacro)
@@ -10,4 +10,5 @@
                 <param name="max">10</param>
             </command_interface>
+            <command_interface name="position" />
             <state_interface name="velocity" />
             <state_interface name="position"/>
@@ -18,4 +19,5 @@
                 <param name="max">10</param>
             </command_interface>
+            <command_interface name="position" />
             <state_interface name="velocity" />
             <state_interface name="position"/>
@@ -26,4 +28,5 @@
                 <param name="max">10</param>
             </command_interface>
+            <command_interface name="position" />
             <state_interface name="velocity" />
             <state_interface name="position"/>
@@ -34,4 +37,41 @@
                 <param name="max">10</param>
             </command_interface>
+            <command_interface name="position" />
+            <state_interface name="velocity" />
+            <state_interface name="position"/>
+        </joint>
+        <joint name="LF_stering_arm_joint">
+            <command_interface name="velocity">
+                <param name="min">-10</param>
+                <param name="max">10</param>
+            </command_interface>
+            <command_interface name="position" />
+            <state_interface name="velocity" />
+            <state_interface name="position"/>
+        </joint>
+        <joint name="RF_stering_arm_joint">
+            <command_interface name="velocity">
+                <param name="min">-10</param>
+                <param name="max">10</param>
+            </command_interface>
+            <command_interface name="position" />
+            <state_interface name="velocity" />
+            <state_interface name="position"/>
+        </joint>
+        <joint name="LR_stering_arm_joint">
+            <command_interface name="velocity">
+                <param name="min">-10</param>
+                <param name="max">10</param>
+            </command_interface>
+            <command_interface name="position" />
+            <state_interface name="velocity" />
+            <state_interface name="position"/>
+        </joint>
+        <joint name="RR_stering_arm_joint">
+            <command_interface name="velocity">
+                <param name="min">-10</param>
+                <param name="max">10</param>
+            </command_interface>
+            <command_interface name="position" />
             <state_interface name="velocity" />
             <state_interface name="position"/>
@@ -40,5 +80,5 @@
     <gazebo>
         <plugin filename="gz_ros2_control-system" name="gz_ros2_control::GazeboSimROS2ControlPlugin">
-            <parameters>$(find sagan_description)/parameters/my_controllers.yaml</parameters>
+            <parameters>$(find sagan_description)/parameters/sagan_controllers_parameters.yaml</parameters>
         </plugin>
     </gazebo>
